File: pcb/cpu.kicad_sch (KiCad schematic)
At the start: 36 parts, among them SW101 EVQPUJ02K, U100 MCIMX6Y7DVM09AB, Y101 24MHz, Y102 32.768kHz

Commit message: pcb: finish routing r0p1
Connections:
- net LCD_EN: now reaches U100.E17 (ENET1_RX_DATA1)
Changed lines of the file:
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@@
+    (stroke (width 0) (type solid) (color 0 0 0 0))
+  )
+  (wire (pts (xy 259.08 198.12) (xy 264.16 198.12))
     (stroke (width 0) (type solid) (color 0 0 0 0))
   )
@@
       (effects (font (size 1.27 1.27)) (justify left) hide)
     )
+  )
+  (global_label "LCD_EN" (shape output) (at 264.16 198.12 0) (fields_autoplaced)
+    (effects (font (size 1.27 1.27)) (justify left))
+    (property "Intersheet References" "${INTERSHEET_REFS}" (id 0) (at 273.5883 198.0406 0)
+      (effects (font (size 1.27 1.27)) (justify left) hide)
+    )

Commit message: pcb: getting ready for r0.2 production
Parts:
- removed C114, C115, C117: 220nF, Capacitor_SMD:C_0402_1005Metric, symbol Device:C
- removed C119: 2.2uF, Capacitor_SMD:C_0402_1005Metric, symbol Device:C
- removed R111: DNP/4.75M, Resistor_SMD:R_0402_1005Metric, symbol Device:R
- removed RN101, RN102, RN103, RN104, RN105, RN106, RN107: 10K, Resistor_SMD:R_Array_Convex_4x0402, symbol Device:R_Pack04
- removed unit 6 of U100
- added SW102: DNP, Button_Switch_SMD:SW_SPST_SKQG_WithStem, symbol Switch:SW_Push
- R101: value 10K -> DNP
- R102: value DNP/10K -> 10K
- R103: value DNP/10K -> DNP
- R109: value 1M -> 2.2M
Connections:
- net CSI_D0 is gone; now on net EPDC_GDSP: U100.B13 (LCD_DATA17)
- net CSI_D1 is gone; now on net EPDC_GDCLK: U100.C13 (LCD_DATA16)
- net CSI_D13 is gone; now on net EPD_TP_INT: U100.B14 (LCD_DATA21)
- net LCD1_CLK is gone; now on net EPDC_SDCLK: U100.A8 (LCD_CLK)
- net LCD1_DE is gone; now on net EPDC_SDLE: U100.B8 (LCD_ENABLE)
- net LCD1_HSYNC is gone; now on net EPDC_SDOE: U100.D9 (LCD_HSYNC)
- net LCD1_RESET is gone; now on net EPDC_GDOE: U100.E9 (LCD_RESET)
- net LCD1_VSYNC is gone; now on net EPDC_SDCE0: U100.C9 (LCD_VSYNC)
- net LCD_D0 is gone; now on net EPDC_D0: U100.B9 (LCD_DATA0)
- net LCD_D1 is gone; now on net EPDC_D1: U100.A9 (LCD_DATA1)
- net LCD_D13 is gone; now on net WL_PMU_EN: U100.B12 (LCD_DATA13)
- net LCD_D14 is gone; now on net WL_WAKE_AP: U100.A12 (LCD_DATA14)
- net LCD_D2 is gone; now on net EPDC_D2: U100.E10 (LCD_DATA2)
- net LCD_D3 is gone; now on net EPDC_D3: U100.D10 (LCD_DATA3)
- net LCD_D4 is gone; now on net EPDC_D4: U100.C10 (LCD_DATA4)
- net LCD_D5 is gone; now on net EPDC_D5: U100.B10 (LCD_DATA5)
- net LCD_D6 is gone; now on net EPDC_D6: U100.A10 (LCD_DATA6)
- net LCD_D7 is gone; now on net EPDC_D7: U100.D11 (LCD_DATA7)
- net +RTC: now also SW102.1
- net EPDC_D0: no longer U100.L14 (GPIO1_IO2)
- net EPDC_D1: no longer U100.L17 (GPIO1_IO3)
- net EPDC_D10: now also U100.B17 (ENET2_RX_EN); no longer U100.M16 (GPIO1_IO4)
- net EPDC_D11: now also U100.A15 (ENET2_TXD0); no longer U100.M17 (GPIO1_IO5)
- net EPDC_D12: now also U100.A16 (ENET2_TXD1); no longer U100.K17 (GPIO1_IO6)
- net EPDC_D13: now also U100.B15 (ENET2_TX_EN); no longer U100.L16 (GPIO1_IO7)
- net EPDC_D14: now also U100.D17 (ENET2_TX_CLK); no longer U100.N17 (GPIO1_IO8)
- net EPDC_D15: now also U100.D16 (ENET2_RX_ER); no longer U100.M15 (GPIO1_IO9)
- net EPDC_D2: no longer U100.K14 (UART1_TX_DATA)
- net EPDC_D3: no longer U100.K16 (UART1_RX_DATA)
- net EPDC_D4: no longer U100.K15 (~{UART1_CTS})
- net EPDC_D5: no longer U100.J14 (~{UART1_RTS})
- net EPDC_D6: no longer U100.J17 (UART2_TX_DATA)
- net EPDC_D7: no longer U100.J16 (UART2_RX_DATA)
- net EPDC_D8: now also U100.C17 (ENET_RX_DATA0); no longer U100.J15 (~{UART1_CTS})
- net EPDC_D9: now also U100.C16 (ENET_RX_DATA1); no longer U100.H14 (~{UART2_RTS})
- net EPDC_GDCLK: no longer U100.R8 (ONOFF)
- net EPDC_GDOE: no longer U100.T9 (SNVS_PMIC_ON_REQ)
- net EPDC_GDSP: no longer R103.1, R104.2, U100.T10 (BOOT_MODE0)
- net EPDC_SDCE0: no longer U100.N10 (SNVS_TAMPER7)
- net EPDC_SDCLK: no longer U100.L15 (GPIO1_IO1)
- net EPDC_SDLE: no longer U100.H17 (UART3_TX_DATA)
- net EPDC_SDOE: no longer U100.H16 (UART3_RX_DATA)
- net EPD_TP_INT: no longer U100.F15 (ENET1_TX_EN)
- net GND: now also R109.1
- net WL_PMU_EN: no longer U100.B5 (~{NAND_CE1})
- net WL_WAKE_AP: no longer U100.E6 (NAND_DQS)
- net at C112.1, U100.T17 (XTALO), Y101.1: no longer R109.2
- net at C113.1, U100.T16 (XTALI), Y101.3: now also R109.2; no longer R109.1
- net QSPI_A_DATA3: now reaches U100.A4 (NAND_CLE)
- net QSPI_A_DATA3: no longer SW101.1
- net USER_BTN: now reaches U100.B4 (NAND_ALE)
- net USER_BTN: now also SW101.1
- net QSPI_A_SCLK: now reaches U100.D5 (~{NAND_WP})
- net EPD_PWR_INT: now reaches U100.R9 (SNVS_TAMPER1)
- net CSI_D10 renamed BT_WAKE
- net CSI_D11: no longer names the net of U100.D14 (LCD_DATA19)
- net CSI_D12: no longer names the net of U100.C14 (LCD_DATA20)
- net CSI_D14 renamed BT_HOST_WAKE
- net CSI_D15: no longer names the net of U100.B16 (LCD_DATA23)
- net EPDC_PWRSTAT: no longer names the net of U100.N8 (SNVS_TAMPER5)
- net LCD_D10: no longer names the net of U100.E12 (LCD_DATA10)
- net LCD_D11: no longer names the net of U100.D12 (LCD_DATA11)
- net LCD_D12: no longer names the net of U100.C12 (LCD_DATA12)
- net LCD_D15: no longer names the net of U100.D13 (LCD_DATA15)
- net LCD_D8: no longer names the net of U100.B11 (LCD_DATA8)
- net LCD_D9 renamed BT_SHUTDOWN
- net LCD_EN: no longer names the net of U100.E17 (ENET1_RX_DATA1)
- net LCD_PWM: no longer names the net of U100.E15 (ENET1_TX_DATA0)
- net SD1_VSELECT: no longer names the net of U100.E16 (ENET1_RX_EN)
- net UART3_RXD renamed QSPI_A_DATA1
- net UART3_TXD renamed QSPI_A_DATA0
- net USB_OTG_ID renamed USB_OTG1_ID
- new net BOOTMODE0: R103.1, R104.2, SW102.2, U100.T10 (BOOT_MODE0)
- new net EPD_PWR_GOOD: U100.J17 (UART2_TX_DATA)
- new net EPD_VCOM_CTRL: U100.J16 (UART2_RX_DATA)
- new net EPD_WAKEUP: U100.K17 (GPIO1_IO6)
- new net PMU_IRQ: U100.N10 (SNVS_TAMPER7)
- new net QSPI_A_DATA2: U100.B5 (~{NAND_CE1})
- new net QSPI_A_SS0: U100.E6 (NAND_DQS)
- new net UART1_RXD: U100.K16 (UART1_RX_DATA)
- new net UART1_TXD: U100.K14 (UART1_TX_DATA)
- new net USB_OTG2_ID: U100.M17 (GPIO1_IO5)
- new net USB_OTG2_OC: U100.L17 (GPIO1_IO3)
- new net USB_OTG2_PWR: U100.L14 (GPIO1_IO2)
- no-connect marks 10 -> 23
Other:
- note removed: "CKV"
- note removed: "MODE"
- note removed: "PWM1"
- note removed: "RFU"
- note removed: "SPV"
- note removed: "XLE"
- note removed: "XOE"
- note removed: "XSTL"
- moved on the sheet: C101, C102, C103, C108, C112, C113, C116, C121, C122, C123, C124, R101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
