File: pcb/ddr.kicad_sch (KiCad schematic)
At the start: 34 parts, among them U100 MCIMX6Y7DVM09AB, U202 MT41K256M16HA

Commit message: pcb: finish routing r0p1
Connections:
- net DRAM_SDQSN_0 is gone; now on net DRAM_LDQSN: U100.P7 (DRAM_SDQS0_N)
- net DRAM_SDQSN_1 is gone; now on net DRAM_UDQSN: U100.T2 (DRAM_SDQS1_N)
- net DRAM_SDQSP_0 is gone; now on net DRAM_LDQSP: U100.P6 (DRAM_SDQS0_P)
- net DRAM_SDQSP_1 is gone; now on net DRAM_UDQSP: U100.T1 (DRAM_SDQS1_P)
- net DRAM_DQM0 renamed DRAM_LDM
- net DRAM_LDM: now also U202.E7 (LDM); no longer U202.D3 (UDM)
- net DRAM_DQM1 renamed DRAM_UDM
- net DRAM_UDM: now also U202.D3 (UDM); no longer U202.E7 (LDM)
Changed lines of the file:
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@@
     (effects (font (size 1.27 1.27)) (justify right bottom))
   )
-  (label "DRAM_SDQSP_0" (at 81.28 93.98 180)
-    (effects (font (size 1.27 1.27)) (justify right bottom))
-  )
-  (label "DRAM_SDQSN_0" (at 81.28 96.52 180)
-    (effects (font (size 1.27 1.27)) (justify right bottom))
-  )
-  (label "DRAM_DQM0" (at 81.28 99.06 180)
+  (label "DRAM_LDQSP" (at 81.28 93.98 180)
+    (effects (font (size 1.27 1.27)) (justify right bottom))
+  )
+  (label "DRAM_LDQSN" (at 81.28 96.52 180)
+    (effects (font (size 1.27 1.27)) (justify right bottom))
+  )
+  (label "DRAM_LDM" (at 81.28 99.06 180)
     (effects (font (size 1.27 1.27)) (justify right bottom))
   )
@@
     (effects (font (size 1.27 1.27)) (justify right bottom))
   )
-  (label "DRAM_SDQSP_1" (at 81.28 124.46 180)
-    (effects (font (size 1.27 1.27)) (justify right bottom))
-  )
-  (label "DRAM_SDQSN_1" (at 81.28 127 180)
-    (effects (font (size 1.27 1.27)) (justify right bottom))
-  )
-  (label "DRAM_DQM1" (at 81.28 129.54 180)
+  (label "DRAM_UDQSP" (at 81.28 124.46 180)
+    (effects (font (size 1.27 1.27)) (justify right bottom))
+  )
+  (label "DRAM_UDQSN" (at 81.28 127 180)
+    (effects (font (size 1.27 1.27)) (justify right bottom))
+  )
+  (label "DRAM_UDM" (at 81.28 129.54 180)
     (effects (font (size 1.27 1.27)) (justify right bottom))
   )
@@
     (effects (font (size 1.27 1.27)) (justify left bottom))
   )
-  (label "DRAM_DQM0" (at 264.16 144.78 0)
-    (effects (font (size 1.27 1.27)) (justify left bottom))
-  )
-  (label "DRAM_DQM1" (at 264.16 147.32 0)
-    (effects (font (size 1.27 1.27)) (justify left bottom))
-  )
+  (label "DRAM_UDM" (at 264.16 144.78 0)
+    (effects (font (size 1.27 1.27)) (justify left bottom))
+  )
+  (label "DRAM_LDM" (at 264.16 147.32 0)
+    (effects (font (size 1.27 1.27)) (justify left bottom))
+  )

Commit message: pcb: getting ready for r0.2 production
Parts:
- added R205: 470, Resistor_SMD:R_0402_1005Metric, symbol Device:R
- U202: footprint footprints:BGA-96_9.0x13.0mm_P0.8mm -> footprints:BGA-96_9.0x14.0mm_P0.8mm
Connections:
- net DRAM_CKN: now also R205.2
- net DRAM_CKP: now also R205.1
Other:
- moved on the sheet: C201, C202, C203, C204, C205, C206, C207, C208, C210, C212, C213, C216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
