File: pcb/lcd.kicad_sch (KiCad schematic)
At the start: 78 parts, among them J501 0.5mm, J502 Conn_01x30_MountingPin, J503 1mm, J504 0.5mm, U501 AP3031, U502 TPS65185, U503 DS90C385A/GM8285C

Commit message: pcb: getting ready for r0.2 production
Parts:
- removed C501: 10uF, Capacitor_SMD:C_0603_1608Metric, symbol Device:C
- removed C503, C512: 100nF, Capacitor_SMD:C_0402_1005Metric, symbol Device:C
- removed C505, C524, C525, C526, C527: 220nF, Capacitor_SMD:C_0402_1005Metric, symbol Device:C
- removed C506: 1uF/35V, Capacitor_SMD:C_0603_1608Metric, symbol Device:C
- removed C520: 10uF/6.3V, Capacitor_SMD:C_0603_1608Metric, symbol Device:C
- removed C528: 22uF, Capacitor_SMD:C_0603_1608Metric, symbol Device:C
- removed D501: B0530WS, Diode_SMD:D_SOD-323, symbol Diode:MBR0530
- removed J502: Conn_01x30_MountingPin, footprints:Hirose_FH12-30S-0.5SH_1x30-1MP_P0.50mm_Horizontal_Reversed, symbol Connector_Generic_MountingPin:Conn_01x30_MountingPin
- removed J504: 0.5mm, footprints:Hirose_FH12-12S-0.5SH_1x12-1MP_P0.50mm_Horizontal_Reversed, symbol Connector_Generic_MountingPin:Conn_01x12_MountingPin
- removed L501: 4.7uH, footprints:L_1212, symbol Device:L
- removed R501: 0R, Resistor_SMD:R_0402_1005Metric, symbol Device:R
- removed R503, R505, R508: 10K, Resistor_SMD:R_0402_1005Metric, symbol Device:R
- removed R504: 49.9K/1%, Resistor_SMD:R_0402_1005Metric, symbol Device:R
- removed R506: 3.3K, Resistor_SMD:R_0402_1005Metric, symbol Device:R
- removed R507: 1.8R, Resistor_SMD:R_0402_1005Metric, symbol Device:R
- removed R516: 100K, Resistor_SMD:R_0402_1005Metric, symbol Device:R
- removed U501: AP3031, Package_TO_SOT_SMD:SOT-23-6, symbol symbols:AP3031
- removed U503: DS90C385A/GM8285C, Package_SO:TSSOP-56_6.1x14mm_P0.5mm, symbol symbols:DS90C385A
- added RN501, RN502, RN503, RN504, RN505, RN506: 33, Resistor_SMD:R_Array_Convex_4x0402, symbol Device:R_Pack04
- J503: value 1mm -> 0.5mm; footprint footprints:Molex_200528-0060_1x06-1MP_P1.00mm_Horizontal_Reversed -> Connector_FFC-FPC:Hirose_FH12-6S-0.5SH_1x06-1MP_P0.50mm_Horizontal
- TH501: footprint Resistor_SMD:R_0402_1005Metric -> Resistor_SMD:R_0603_1608Metric
Connections:
- net BORDER is gone; now on net VCOM: C502.1, J501.40 (Pin_40)
- net I2C_SCL is gone; now on net I2C1_SCL: U502.17 (SCL)
- net I2C_SDA is gone; now on net I2C1_SDA: U502.18 (SDA)
- net EPDC_D0: now also RN502.6 (R3.2); no longer J501.14 (Pin_14)
- net EPDC_D1: now also RN502.7 (R2.2); no longer J501.15 (Pin_15)
- net EPDC_D10: now also RN504.8 (R1.2); no longer J501.25 (Pin_25)
- net EPDC_D11: now also RN505.5 (R4.2); no longer J501.26 (Pin_26)
- net EPDC_D12: now also RN505.6 (R3.2); no longer J501.27 (Pin_27)
- net EPDC_D13: now also RN505.7 (R2.2); no longer J501.28 (Pin_28)
- net EPDC_D14: now also RN505.8 (R1.2); no longer J501.29 (Pin_29)
- net EPDC_D15: now also RN506.5 (R4.2); no longer J501.30 (Pin_30)
- net EPDC_D2: now also RN502.8 (R1.2); no longer J501.16 (Pin_16)
- net EPDC_D3: now also RN503.5 (R4.2); no longer J501.17 (Pin_17)
- net EPDC_D4: now also RN503.6 (R3.2); no longer J501.18 (Pin_18)
- net EPDC_D5: now also RN503.7 (R2.2); no longer J501.19 (Pin_19)
- net EPDC_D6: now also RN503.8 (R1.2); no longer J501.20 (Pin_20)
- net EPDC_D7: now also RN504.5 (R4.2); no longer J501.21 (Pin_21)
- net EPDC_D8: now also RN504.6 (R3.2); no longer J501.23 (Pin_23)
- net EPDC_D9: now also RN504.7 (R2.2); no longer J501.24 (Pin_24)
- net EPDC_GDCLK: now also RN501.7 (R2.2); no longer J501.7 (Pin_7)
- net EPDC_GDOE: now also RN501.6 (R3.2); no longer J501.6 (Pin_6)
- net EPDC_GDSP: now also RN501.8 (R1.2); no longer J501.8 (Pin_8)
- net EPDC_SDCE0: now also RN506.6 (R3.2); no longer J501.31 (Pin_31)
- net EPDC_SDCLK: now also RN502.5 (R4.2); no longer J501.13 (Pin_13)
- net EPDC_SDLE: now also RN506.7 (R2.2); no longer J501.32 (Pin_32)
- net EPDC_SDOE: now also RN506.8 (R1.2); no longer J501.33 (Pin_33)
- net VN: now reaches C532.1, C535.1, C536.1, D506.1 (K), U502.16 (VCOM_PWR), U502.22 (PBKG), U502.26 (VN), U502.27 (VEE_IN), U502.4 (VNEG_IN), U502.49 (EP)
- net VP: now reaches C521.2, C523.2, D504.1 (K), U502.37 (VDDH_IN), U502.42 (VB), U502.43 (VPOS_IN)
- net EPD_PWR_INT: now reaches U502.2 (~{INT})
- net EPD_WAKEUP: now reaches U502.5 (WAKEUP)
- net EPDC_BDR0 renamed EPD_VCOM_CTRL
- net EPD_PWROK renamed EPD_PWR_GOOD
- new net: J501.13 (Pin_13), RN502.4 (R4.1)
- new net: J501.14 (Pin_14), RN502.3 (R3.1)
- new net: J501.15 (Pin_15), RN502.2 (R2.1)
- new net: J501.16 (Pin_16), RN502.1 (R1.1)
- new net: J501.17 (Pin_17), RN503.4 (R4.1)
- new net: J501.18 (Pin_18), RN503.3 (R3.1)
- new net: J501.19 (Pin_19), RN503.2 (R2.1)
- new net: J501.20 (Pin_20), RN503.1 (R1.1)
- new net: J501.21 (Pin_21), RN504.4 (R4.1)
- new net: J501.23 (Pin_23), RN504.3 (R3.1)
- new net: J501.24 (Pin_24), RN504.2 (R2.1)
- new net: J501.25 (Pin_25), RN504.1 (R1.1)
- new net: J501.26 (Pin_26), RN505.4 (R4.1)
- new net: J501.27 (Pin_27), RN505.3 (R3.1)
- new net: J501.28 (Pin_28), RN505.2 (R2.1)
- new net: J501.29 (Pin_29), RN505.1 (R1.1)
- new net: J501.30 (Pin_30), RN506.4 (R4.1)
- new net: J501.31 (Pin_31), RN506.3 (R3.1)
- new net: J501.32 (Pin_32), RN506.2 (R2.1)
- new net: J501.33 (Pin_33), RN506.1 (R1.1)
- new net: J501.6 (Pin_6), RN501.3 (R3.1)
- new net: J501.7 (Pin_7), RN501.2 (R2.1)
- new net: J501.8 (Pin_8), RN501.1 (R1.1)
- no-connect marks 23 -> 6
Other:
- note removed: "DDC"
- moved on the sheet: C502, C504, C507, C508, C510, C511, C513, C514, C515, C516, C517, C518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
