File: pcb/pcb.kicad_sch (KiCad schematic)
At the start: 0 parts

Commit message: pcb: getting ready for r0.2 production
Other:
- removed sheet audio
- removed sheet dvp
- removed sheet ethernet
- added sheet expansion (expansion.kicad_sch)
- note added: "0.1 2021-09"
- note added: "0.2 2021-09"
- note added: "1. Fixed EPD pinmux 2. Fixed EPD power supply signal connections 3. Removed audio codec 4. Replaced RL-SM02BD with AP6330/6212 5. Removed LCD connector 6. Enabled OTG on one USB port with current limit 7. Replaced CP2102 with CH340 8. Fixed DDR PHY power supply issue 9. Added QSPI NOR to allow SD-less operation 10. Enabled SDR104 operation on SD card 11. Added additional DDR clock termination 12.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"
- note added: "1. Initial release"
- note added: "Expansion"
- note added: "Rev Date Description"
- note added: "Revision History"
- note removed: "8"
- note removed: "9"
- note removed: "Audio"
- note removed: "Ethernet"
- note removed: "Video Input"
