File: pcb/mainboard/expansion.kicad_sch (KiCad schematic)
At the start: 1 part, among them J300 Conn_02x09_Odd_Even

Commit message: pcb: switch to max17135, length tuning for QSPI and SD
Connections:
- net IPSOUT is gone; now on net +3V3: J300.4 (Pin_4)
Changed lines of the file:
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@@
     (pin "1")
   )
-  (symbol (lib_id "symbols:IPSOUT") (at 154.94 96.52 270) (mirror x) (unit 1)
+  (symbol (lib_id "power:+3V3") (at 154.94 96.52 270) (unit 1)
     (in_bom yes) (on_board yes)
     (property "Reference" "#PWR0117" (id 0) (at 151.13 96.52 0)
       (effects (font (size 1.27 1.27)) hide)
     )
-    (property "Value" "IPSOUT" (id 1) (at 161.8742 96.0882 90))
+    (property "Value" "+3V3" (id 1) (at 158.1912 96.266 90)
+      (effects (font (size 1.27 1.27)) (justify left))
+    )
     (property "Footprint" "" (id 2) (at 154.94 96.52 0)
       (effects (font (size 1.27 1.27)) hide)
